File: WormDriver.sch (KiCad schematic (older format))
At the start: 10 parts, among them U8 DRV8424E

Commit message: Finished routing
Parts:
- removed C26: 100uF, Capacitor_SMD:C_0402_1005Metric, symbol Device:C_Small
- added C26: 100uF, Capacitor_Tantalum_SMD:CP_EIA-3528-15_AVX-H_Pad1.50x2.35mm_HandSolder, symbol Device:CP1_Small
Connections:
- net +5V: now also C26.1
- net GND: now also C26.2
Changed lines of the file:
@@
 	1    0    0    -1
 $EndComp
-$Comp
-L Device:C_Small C26
-U 1 1 6173ACFE
-P 5050 3950
-F 0 "C26" H 4900 4000 50  0000 L CNN
-F 1 "100uF" H 4750 3900 50  0000 L CNN
-F 2 "Capacitor_SMD:C_0402_1005Metric" H 5050 3950 50  0001 C CNN
-F 3 "~" H 5050 3950 50  0001 C CNN
-	1    5050 3950
-	1    0    0    -1
-$EndComp
 Wire Wire Line
 	5050 4050 5400 4050
@@
 	1    0    0    -1
 $EndComp
-Connection ~ 5050 4050
 $Comp
 L power:+5V #PWR052
@@
 Wire Wire Line
 	5050 3850 5400 3850
-Connection ~ 5050 3850
 Connection ~ 5400 3850
 Wire Wire Line
@@
 Text Notes 1650 2350 0    591  ~ 118
 Worm Motor Driver
+$Comp
+L Device:CP1_Small C26
+U 1 1 61830E33
+P 5050 3950
+F 0 "C26" H 4850 4000 50  0000 L CNN
+F 1 "100uF" H 4800 3900 50  0000 L CNN
+F 2 "Capacitor_Tantalum_SMD:CP_EIA-3528-15_AVX-H_Pad1.50x2.35mm_HandSolder" H 5050 3950 50  0001 C CNN
+F 3 "~" H 5050 3950 50  0001 C CNN
+	1    5050 3950
+	1    0    0    -1
+$EndComp
+Connection ~ 5050 3850
+Connection ~ 5050 4050
 $EndSCHEMATC
