File: WormDriver.sch (KiCad schematic (older format))
At the start: 10 parts, among them U8 DRV8424E

Commit message: Changes made
Parts:
- renumbered C25 to C23, C26 to C24, C27 to C25, C28 to C26, C29 to C27, C30 to C28, U8 to U7
Changed lines of the file:
@@
 $EndDescr
 $Comp
-L Device:C_Small C28
+L Device:C_Small C26
 U 1 1 6172118F
 P 7550 4100
-F 0 "C28" H 7642 4146 50  0000 L CNN
+F 0 "C26" H 7642 4146 50  0000 L CNN
 F 1 "0.022uF" H 7642 4055 50  0000 L CNN
 F 2 "Capacitor_SMD:C_0402_1005Metric" H 7550 4100 50  0001 C CNN
@@
 VCP
 $Comp
-L Device:C_Small C30
+L Device:C_Small C28
 U 1 1 617225A7
 P 8350 4200
-F 0 "C30" V 8250 4250 50  0000 L CNN
+F 0 "C28" V 8250 4250 50  0000 L CNN
 F 1 "0.22uF" V 8400 4250 50  0000 L CNN
 F 2 "Capacitor_SMD:C_0402_1005Metric" H 8350 4200 50  0001 C CNN
@@
 $EndComp
 $Comp
-L power:GND #PWR051
+L power:GND #PWR045
 U 1 1 6172878B
 P 8800 3650
-F 0 "#PWR051" H 8800 3400 50  0001 C CNN
+F 0 "#PWR045" H 8800 3400 50  0001 C CNN
 F 1 "GND" H 8805 3477 50  0000 C CNN
 F 2 "" H 8800 3650 50  0001 C CNN
@@
 $EndComp
 $Comp
-L power:GND #PWR058
+L power:GND #PWR052
 U 1 1 61728F37
 P 6250 4550
-F 0 "#PWR058" H 6250 4300 50  0001 C CNN
+F 0 "#PWR052" H 6250 4300 50  0001 C CNN
 F 1 "GND" H 6255 4377 50  0000 C CNN
 F 2 "" H 6250 4550 50  0001 C CNN
@@
 	6250 3950 6250 4550
 $Comp
-L Device:C_Small C29
+L Device:C_Small C27
 U 1 1 61737F80
 P 5650 4150
-F 0 "C29" H 5500 4200 50  0000 L CNN
+F 0 "C27" H 5500 4200 50  0000 L CNN
 F 1 "0.47uF" H 5300 4100 50  0000 L CNN
 F 2 "Capacitor_SMD:C_0402_1005Metric" H 5650 4150 50  0001 C CNN
@@
 $EndComp
 $Comp
-L power:GND #PWR056
+L power:GND #PWR050
 U 1 1 617391F8
 P 5650 4250
-F 0 "#PWR056" H 5650 4000 50  0001 C CNN
+F 0 "#PWR050" H 5650 4000 50  0001 C CNN
 F 1 "GND" H 5655 4077 50  0000 C CNN
 F 2 "" H 5650 4250 50  0001 C CNN
@@
 $EndComp
 $Comp
-L Device:C_Small C27
+L Device:C_Small C25
 U 1 1 61739FDA
 P 5400 3950
-F 0 "C27" H 5250 4000 50  0000 L CNN
+F 0 "C25" H 5250 4000 50  0000 L CNN
 F 1 "0.01uF" H 5100 3900 50  0000 L CNN
 F 2 "Capacitor_SMD:C_0402_1005Metric" H 5400 3950 50  0001 C CNN
@@
 	5050 4050 5400 4050
 $Comp
-L power:GND #PWR054
+L power:GND #PWR048
 U 1 1 6173D2DF
 P 5050 4050
-F 0 "#PWR054" H 5050 3800 50  0001 C CNN
+F 0 "#PWR048" H 5050 3800 50  0001 C CNN
 F 1 "GND" H 5055 3877 50  0000 C CNN
 F 2 "" H 5050 4050 50  0001 C CNN
@@
 $EndComp
 $Comp
-L power:+5V #PWR052
+L power:+5V #PWR046
 U 1 1 6173D637
 P 5050 3850
-F 0 "#PWR052" H 5050 3700 50  0001 C CNN
+F 0 "#PWR046" H 5050 3700 50  0001 C CNN
 F 1 "+5V" H 4950 3950 50  0000 C CNN
 F 2 "" H 5050 3850 50  0001 C CNN
@@
 	5400 3850 5650 3850
 $Comp
-L power:GND #PWR050
+L power:GND #PWR044
 U 1 1 6174BC11
 P 7950 3450
-F 0 "#PWR050" H 7950 3200 50  0001 C CNN
+F 0 "#PWR044" H 7950 3200 50  0001 C CNN
 F 1 "GND" H 7955 3277 50  0000 C CNN
 F 2 "" H 7950 3450 50  0001 C CNN
@@
 WORM1_DIR
 $Comp
-L power:+5V #PWR053
+L power:+5V #PWR047
 U 1 1 6174E312
 P 7950 3950
-F 0 "#PWR053" H 7950 3800 50  0001 C CNN
+F 0 "#PWR047" H 7950 3800 50  0001 C CNN
 F 1 "+5V" H 7965 4123 50  0000 C CNN
 F 2 "" H 7950 3950 50  0001 C CNN
@@
 	5750 3350 5900 3350
 $Comp
-L power:GND #PWR049
+L power:GND #PWR043
 U 1 1 61725219
 P 5750 3350
-F 0 "#PWR049" H 5750 3100 50  0001 C CNN
+F 0 "#PWR043" H 5750 3100 50  0001 C CNN
 F 1 "GND" H 5755 3177 50  0000 C CNN
 F 2 "" H 5750 3350 50  0001 C CNN
@@
 $EndComp
 $Comp
-L Device:C_Small C25
+L Device:C_Small C23
 U 1 1 61723FFB
 P 5750 3250
-F 0 "C25" H 5600 3300 50  0000 L CNN
+F 0 "C23" H 5600 3300 50  0000 L CNN
 F 1 "0.01uF" H 5400 3200 50  0000 L CNN
 F 2 "Capacitor_SMD:C_0402_1005Metric" H 5750 3250 50  0001 C CNN
@@
 $EndBitmap
 $Comp
-L power:+5V #PWR048
+L power:+5V #PWR042
 U 1 1 6172F1EA
 P 8800 3150
-F 0 "#PWR048" H 8800 3000 50  0001 C CNN
+F 0 "#PWR042" H 8800 3000 50  0001 C CNN
 F 1 "+5V" H 8700 3250 50  0000 C CNN
 F 2 "" H 8800 3150 50  0001 C CNN
@@
 $EndComp
 $Comp
-L power:+5V #PWR047
+L power:+5V #PWR041
 U 1 1 6189F605
 P 5750 3150
-F 0 "#PWR047" H 5750 3000 50  0001 C CNN
+F 0 "#PWR041" H 5750 3000 50  0001 C CNN
 F 1 "+5V" H 5650 3250 50  0000 C CNN
 F 2 "" H 5750 3150 50  0001 C CNN
@@
 	5750 3150 6350 3150
 $Comp
-L power:+5V #PWR055
+L power:+5V #PWR049
 U 1 1 6183B245
 P 8250 4200
-F 0 "#PWR055" H 8250 4050 50  0001 C CNN
+F 0 "#PWR049" H 8250 4050 50  0001 C CNN
 F 1 "+5V" H 8150 4300 50  0000 C CNN
 F 2 "" H 8250 4200 50  0001 C CNN
@@
 nSLEEP
 $Comp
-L power:GND #PWR057
+L power:GND #PWR051
 U 1 1 61840BB8
 P 7350 4350
-F 0 "#PWR057" H 7350 4100 50  0001 C CNN
+F 0 "#PWR051" H 7350 4100 50  0001 C CNN
 F 1 "GND" H 7355 4177 50  0000 C CNN
 F 2 "" H 7350 4350 50  0001 C CNN
@@
 $EndComp
 $Comp
-L Driver_Motor:DRV8424E U8
+L Driver_Motor:DRV8424E U7
 U 1 1 61885D44
 P 6850 3700
-F 0 "U8" H 6850 4515 50  0000 C CNN
+F 0 "U7" H 6850 4515 50  0000 C CNN
 F 1 "DRV8424E" H 6850 4424 50  0000 C CNN
 F 2 "Package_DFN_QFN:VQFN-24-1EP_4x4mm_P0.5mm_EP2.45x2.45mm" H 6850 2950 50  0001 C CNN
@@
 Worm Motor Driver
 $Comp
-L Device:CP1_Small C26
+L Device:CP1_Small C24
 U 1 1 61830E33
 P 5050 3950
-F 0 "C26" H 4850 4000 50  0000 L CNN
+F 0 "C24" H 4850 4000 50  0000 L CNN
 F 1 "100uF" H 4800 3900 50  0000 L CNN
 F 2 "Capacitor_Tantalum_SMD:CP_EIA-3528-15_AVX-H_Pad1.50x2.35mm_HandSolder" H 5050 3950 50  0001 C CNN
