File: Autodrone.sch (KiCad schematic (older format))
At the start: 7 parts

Commit message: Lots of changes made
Parts:
- removed L3: USN, Footprints:USN, symbol Logos:USN
- renumbered L4 to L2, L5 to L3
Connections:
- net labels added: WORM1_H, WORM1_L, WORM2_H, WORM2_L
- wire segments 45 -> 49
Other:
- moved on the sheet: H1, H2, H3, H4

Commit message: Changes made
Parts:
- added L5, L6: LED, Footprints:LED, symbol Logos:LED
- renumbered L2 to L1, L3 to L2
Changed lines of the file:
@@
 F0 "Gyro" 59
 F1 "Gyro.sch" 59
-F2 "SPI1_MOSI" I L 5350 3200 50
-F3 "SPI1_MISO" I L 5350 3100 50
-F4 "SPI1_SCK" I L 5350 3000 50
-F5 "SPI1_CS" I L 5350 2900 50
+F2 "SPI1_MOSI" I L 5350 2900 50
+F3 "SPI1_MISO" I L 5350 3000 50
+F4 "SPI1_SCK" I L 5350 3100 50
+F5 "SPI1_CS" I L 5350 3200 50
 $EndSheet
 $Sheet
@@
 VID
 $Comp
-L Logos:EGA L2
+L Logos:EGA L1
 U 1 1 60A40993
 P 6950 6000
-F 0 "L2" H 6975 6046 50  0000 L CNN
+F 0 "L1" H 6975 6046 50  0000 L CNN
 F 1 "EGA" H 6975 5955 50  0000 L CNN
 F 2 "Footprints:EGA" H 6950 6000 50  0001 C CNN
@@
 $EndComp
 $Comp
-L Logos:Arrow L3
+L Logos:Arrow L2
 U 1 1 60A46BB1
 P 7150 6000
-F 0 "L3" H 7175 6046 50  0000 L CNN
+F 0 "L2" H 7175 6046 50  0000 L CNN
 F 1 "Arrow" H 7175 5955 50  0000 L CNN
 F 2 "Footprints:Arrow" H 7150 6000 50  0001 C CNN
@@
 Wire Wire Line
 	3950 4200 4100 4200
+$Comp
+L Logos:LED L5
+U 1 1 61932C41
+P 7400 6000
+F 0 "L5" H 7425 6046 50  0000 L CNN
+F 1 "LED" H 7425 5955 50  0000 L CNN
+F 2 "Footprints:LED" H 7400 6000 50  0001 C CNN
+F 3 "" H 7400 6000 50  0001 C CNN
+	1    7400 6000
+	1    0    0    -1
+$EndComp
+$Comp
+L Logos:LED L6
+U 1 1 61933AF3
+P 7600 6000
+F 0 "L6" H 7625 6046 50  0000 L CNN
+F 1 "LED" H 7625 5955 50  0000 L CNN
+F 2 "Footprints:LED" H 7600 6000 50  0001 C CNN
+F 3 "" H 7600 6000 50  0001 C CNN
+	1    7600 6000
+	1    0    0    -1
+$EndComp
 $EndSCHEMATC
