File: Debugger.sch (KiCad schematic (older format))
At the start: 1 part, among them U9 STLINK-V3MODS

Commit message: Changes made
Parts:
- renumbered U9 to U8
Changed lines of the file:
@@
 $EndDescr
 $Comp
-L JPW_Symbols:STLINK-V3MODS U9
+L JPW_Symbols:STLINK-V3MODS U8
 U 1 1 616F1D27
 P 6350 3350
-F 0 "U9" H 7375 3615 50  0000 C CNN
+F 0 "U8" H 7375 3615 50  0000 C CNN
 F 1 "STLINK-V3MODS" H 7375 3524 50  0000 C CNN
 F 2 "Footprints:STLINKV3MODS" H 8650 3550 50  0001 L BNN
@@
 	6350 4050 6350 4950
 $Comp
-L power:GND #PWR060
+L power:GND #PWR054
 U 1 1 616F42B7
 P 6350 4950
-F 0 "#PWR060" H 6350 4700 50  0001 C CNN
+F 0 "#PWR054" H 6350 4700 50  0001 C CNN
 F 1 "GND" H 6355 4777 50  0000 C CNN
 F 2 "" H 6350 4950 50  0001 C CNN
@@
 $EndComp
 $Comp
-L power:GND #PWR061
+L power:GND #PWR055
 U 1 1 616F4B84
 P 8400 4950
-F 0 "#PWR061" H 8400 4700 50  0001 C CNN
+F 0 "#PWR055" H 8400 4700 50  0001 C CNN
 F 1 "GND" H 8405 4777 50  0000 C CNN
 F 2 "" H 8400 4950 50  0001 C CNN
@@
 NRST
 $Comp
-L power:+3V3 #PWR059
+L power:+3V3 #PWR053
 U 1 1 617F4C8C
 P 8700 3500
-F 0 "#PWR059" H 8700 3350 50  0001 C CNN
+F 0 "#PWR053" H 8700 3350 50  0001 C CNN
 F 1 "+3V3" H 8715 3673 50  0000 C CNN
 F 2 "" H 8700 3500 50  0001 C CNN
