File: MCU.sch (KiCad schematic (older format))
At the start: 36 parts, among them Q1 BSS138, SW1 SW_Push, U2 STM32F722RETx

Commit message: Lots of changes made
Parts:
- removed C26, C32: 10pF, Capacitor_SMD:C_0402_1005Metric, symbol Device:C_Small
- removed HSE1: 8MHz, Oscillator:Oscillator_SMD_Abracon_ASE-4Pin_3.2x2.5mm, symbol Device:Crystal_GND24_Small
- added D11: GREEN, LED_SMD:LED_0603_1608Metric, symbol Device:LED_Small
- added D5: BLUE, LED_SMD:LED_0603_1608Metric, symbol Device:LED_Small
- added D7: RED, LED_SMD:LED_0603_1608Metric, symbol Device:LED_Small
- added D9: YELLOW, LED_SMD:LED_0603_1608Metric, symbol Device:LED_Small
- added JP1, JP2: SolderJumper_2_Open, Jumper:SolderJumper-2_P1.3mm_Open_TrianglePad1.0x1.5mm, symbol Jumper:SolderJumper_2_Open
- added R27, R31, R33, R35: 1k, Resistor_SMD:R_0402_1005Metric, symbol Device:R_Small
- added Y2: CSTNE8M00G55Z000R0, Footprints:OSC_CSTNE8M00G55Z000R0, symbol JPW_Symbols:CSTNE8M00G55Z000R0
- R25: renamed from R6; value 2k -> 330
- R34: renamed from R26; value 100 -> 1k
- R36: renamed from R28; value 233 -> 1k
- renumbered C13 to C39, C14 to C40, C3 to C41, C4 to C42, C5 to C43, C6 to C44, C7 to C45, C8 to C46, C15 to C47, C11 to C48, D7 to D10, D8 to D12, D9 to D13, D5 to D6, D3 to D8, FB2 to FB3, R27 to R20, R31 to R21, R2 to R22, R3 to R23, R4 to R24, R1 to R26, R23 to R28, R7 to R29, R15 to R30, R21 to R32, R9 to R37, U2 to U11
Connections:
- net LED is gone; now on net M2: U11.15 (PA1)
- net UART2_RX is gone; now on net M4: U11.17 (PA3)
- net UART2_TX is gone; now on net M3: U11.16 (PA2)
- net GND: now also R27.2, R31.2, R33.2, R35.2, Y2.2
- net HSE_IN: now also Y2.1
- net I2C1_SCL: now also U11.61 (PB8); no longer R24.2, U11.58 (PB6)
- net I2C1_SDA: now also U11.62 (PB9); no longer R23.2, U11.59 (PB7)
- net M1: now also U11.14 (PA0); no longer U11.26 (PB1)
- net M2: no longer U11.25 (PB0)
- net M3: no longer U11.57 (PB5)
- net M4: no longer U11.56 (PB4)
- net 9V: now reaches D12.1 (K), R36.1
- net 5V: now reaches D10.1 (K), R34.1
- net at R25.2: now also Y2.3
- net 1V8: now reaches D6.1 (K), R28.1
- net 3V3: now reaches D8.1 (K), R32.1
- net LED_4: now reaches U11.11 (PC3)
- net LED_4: now also D11.2 (A)
- net LIMIT1_INT: now reaches U11.2 (PC13)
- net LIMIT2_INT: now reaches U11.3 (PC14)
- net VCAP: now reaches C48.1, U11.30 (VCAP_1)
- net WORM1_DIR: now reaches U11.39 (PC8)
- net UART5_RX: now reaches U11.54 (PD2)
- net UART5_RX: now also JP1.1 (A)
- net LED_2: now reaches U11.9 (PC1)
- net LED_2: now also D7.2 (A)
- net +VCC: now reaches D13.1 (K), R37.1
- net ADC_VSENS renamed VCC_SENSE
- net VCC_SENSE: now also U11.25 (PB0); no longer U11.10 (PC2)
- net BUZ- renamed BUZ
- net BUZ-_MCU renamed BUZ_MCU
- net BUZ_MCU: now also U11.57 (PB5); no longer U11.24 (PC4)
- net CURR renamed LED_1
- net LED_1: now also D5.2 (A)
- net I2C3_SCL renamed WORM1_PWM
- net I2C3_SDA renamed WORM2_DIR
- net LED_BLUE renamed +1V8
- net +1V8: no longer U11.14 (PA0)
- net SPI3_CS: no longer names the net of U11.50 (PA15)
- net SPI3_MISO renamed USART3_RX
- net SPI3_MOSI renamed UART5_TX
- net UART5_TX: now also JP2.1 (A)
- net SPI3_SCK renamed USART3_TX
- net UART1_RX: no longer names the net of U11.43 (PA10)
- net UART1_TX renamed WORM2_PWM
- net UART3_RX renamed I2C2_SDA
- net I2C2_SDA: now also R23.2
- net UART3_TX renamed I2C2_SCL
- net I2C2_SCL: now also R24.2
- net UART6_RX renamed USART6_RX
- net UART6_TX renamed USART6_TX
- new net ADC: U11.24 (PC4)
- new net BLUE: D5.1 (K), R27.1
- new net CURR_SENSE: U11.26 (PB1)
- new net GREEN: D11.1 (K), R35.1
- new net LED_3: D9.2 (A), U11.10 (PC2)
- new net LED_STRIP: U11.56 (PB4)
- new net RED: D7.1 (K), R31.1
- new net UART5_RX_CONN: JP1.2 (B)
- new net UART5_TX_CONN: JP2.2 (B)
- new net USART1_RX: U11.59 (PB7)
- new net USART1_TX: U11.58 (PB6)
- new net YELLOW: D9.1 (K), R33.1
- no-connect marks 9 -> 4
Other:
- note added: "Power LEDs"
- note added: "User LEDs"
- note removed: "LEDs"
- moved on the sheet: C39, C40, C47, D10, D12, D13, D6, D8, FB3, Q1, R22, R25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

Commit message: Finished routing
Parts:
- R23, R24: value 3.7k -> 2k2
Connections:
- net BUZ_MCU: now also U11.56 (PB4); no longer U11.57 (PB5)
- net LED_STRIP: now also U11.57 (PB5); no longer U11.56 (PB4)
- net M1: now also U11.17 (PA3); no longer U11.14 (PA0)
- net M2: now also U11.16 (PA2); no longer U11.15 (PA1)
- net M3: now also U11.15 (PA1); no longer U11.16 (PA2)
- net M4: now also U11.14 (PA0); no longer U11.17 (PA3)
Changed lines of the file:
@@
 P 9700 2650
 F 0 "R23" V 9700 2600 50  0000 L CNN
-F 1 "3.7k" V 9600 2550 50  0000 L CNN
+F 1 "2k2" V 9600 2550 50  0000 L CNN
 F 2 "Resistor_SMD:R_0402_1005Metric" H 9700 2650 50  0001 C CNN
 F 3 "~" H 9700 2650 50  0001 C CNN
@@
 P 9700 2900
 F 0 "R24" V 9700 2850 50  0000 L CNN
-F 1 "3.7k" V 9600 2800 50  0000 L CNN
+F 1 "2k2" V 9600 2800 50  0000 L CNN
 F 2 "Resistor_SMD:R_0402_1005Metric" H 9700 2900 50  0001 C CNN
 F 3 "~" H 9700 2900 50  0001 C CNN
@@
 Wire Wire Line
 	6150 2650 6550 2650
-Text HLabel 6350 3900 2    50   Input ~ 0
+Text HLabel 6350 4000 2    50   Input ~ 0
 M2
 $Comp
@@
 Text HLabel 6350 6700 2    50   Input ~ 0
 SPI2_CS
-Text HLabel 6350 3800 2    50   Input ~ 0
-M1
 Text HLabel 6350 4100 2    50   Input ~ 0
+M1
+Text HLabel 6350 3800 2    50   Input ~ 0
 M4
-Text HLabel 6350 4000 2    50   Input ~ 0
+Text HLabel 6350 3900 2    50   Input ~ 0
 M3
 Text HLabel 6350 4200 2    50   Input ~ 0
@@
 Text Label 5050 5900 2    50   ~ 0
 LED_4
-Text HLabel 6350 5900 2    50   Input ~ 0
+Text HLabel 6350 6000 2    50   Input ~ 0
 LED_STRIP
 NoConn ~ 6350 4800
-Text Label 6350 6000 0    50   ~ 0
+Text Label 6350 5900 0    50   ~ 0
 BUZ_MCU
 Text HLabel 5050 6000 0    50   Input ~ 0

Commit message: Changes made
Parts:
- renumbered C39 to C37, C40 to C38, C41 to C39, C42 to C40, C43 to C41, C44 to C42, C45 to C43, C46 to C44, C47 to C45, C48 to C46, U11 to U10
Connections:
- net +1V8 renamed +3V3_GYRO
- net 1V8 renamed 3V3_GYRO
