File: OSD.sch (KiCad schematic (older format))
At the start: 16 parts, among them U6 MAX7456EUI+, Y1 27MHz

Commit message: Lots of changes made
Parts:
- renumbered C37 to C31, C38 to C32, C39 to C33, C40 to C34, C41 to C35, C42 to C36, C43 to C37, C44 to C38, R25 to R14, R29 to R15, R30 to R16, R33 to R17, R34 to R18, R35 to R19, U6 to U10
Connections:
- net LOS: now reaches R16.2, U10.12 (LOS)
- net LSYNC: now reaches R15.2, U10.17 (~VSYNC)
- net HSYNC: now reaches R14.2, U10.18 (~HSYNC)
- net VIN: now reaches C33.2, U10.22 (VIN)
- net VOUT: now reaches C31.2, U10.26 (VOUT)
Changed lines of the file:
@@
 $Descr A4 11693 8268
 encoding utf-8
-Sheet 5 8
+Sheet 7 9
 Title ""
 Date ""
@@
 P 7200 4850
 AR Path="/60B200F8" Ref="C?"  Part="1"
-AR Path="/60B17C6E/60B200F8" Ref="C43"  Part="1"
-F 0 "C43" H 7350 4800 50  0000 R CNN
+AR Path="/60B17C6E/60B200F8" Ref="C37"  Part="1"
+F 0 "C37" H 7350 4800 50  0000 R CNN
 F 1 "10pF" H 7500 4900 50  0000 R CNN
 F 2 "Capacitor_SMD:C_0402_1005Metric" H 7200 4850 50  0001 C CNN
@@
 P 7600 4850
 AR Path="/60B20102" Ref="C?"  Part="1"
-AR Path="/60B17C6E/60B20102" Ref="C44"  Part="1"
-F 0 "C44" H 7550 4800 50  0000 R CNN
+AR Path="/60B17C6E/60B20102" Ref="C38"  Part="1"
+F 0 "C38" H 7550 4800 50  0000 R CNN
 F 1 "10pF" H 7500 4900 50  0000 R CNN
 F 2 "Capacitor_SMD:C_0402_1005Metric" H 7600 4850 50  0001 C CNN
@@
 P 7350 4950
 AR Path="/60B2010C" Ref="#PWR?"  Part="1"
-AR Path="/60B17C6E/60B2010C" Ref="#PWR0157"  Part="1"
-F 0 "#PWR0157" H 7350 4700 50  0001 C CNN
+AR Path="/60B17C6E/60B2010C" Ref="#PWR069"  Part="1"
+F 0 "#PWR069" H 7350 4700 50  0001 C CNN
 F 1 "GND" H 7355 4777 50  0000 C CNN
 F 2 "" H 7350 4950 50  0001 C CNN
@@
 P 7700 4650
 AR Path="/60B2011A" Ref="R?"  Part="1"
-AR Path="/60B17C6E/60B2011A" Ref="R35"  Part="1"
-F 0 "R35" V 7504 4650 50  0000 C CNN
+AR Path="/60B17C6E/60B2011A" Ref="R19"  Part="1"
+F 0 "R19" V 7504 4650 50  0000 C CNN
 F 1 "589" V 7595 4650 50  0000 C CNN
 F 2 "Resistor_SMD:R_0402_1005Metric" H 7700 4650 50  0001 C CNN
@@
 P 8550 4650
 AR Path="/60B20121" Ref="C?"  Part="1"
-AR Path="/60B17C6E/60B20121" Ref="C40"  Part="1"
-F 0 "C40" H 8400 4550 50  0000 C CNN
+AR Path="/60B17C6E/60B20121" Ref="C34"  Part="1"
+F 0 "C34" H 8400 4550 50  0000 C CNN
 F 1 "0.1uF" H 8650 4700 50  0000 C CNN
 F 2 "Capacitor_SMD:C_0402_1005Metric" H 8550 4650 50  0001 C CNN
@@
 P 8850 4650
 AR Path="/60B20127" Ref="C?"  Part="1"
-AR Path="/60B17C6E/60B20127" Ref="C41"  Part="1"
-F 0 "C41" H 8750 4550 50  0000 C CNN
+AR Path="/60B17C6E/60B20127" Ref="C35"  Part="1"
+F 0 "C35" H 8750 4550 50  0000 C CNN
 F 1 "0.1uF" H 9000 4700 50  0000 C CNN
 F 2 "Capacitor_SMD:C_0402_1005Metric" H 8850 4650 50  0001 C CNN
@@
 P 9150 4650
 AR Path="/60B20133" Ref="C?"  Part="1"
-AR Path="/60B17C6E/60B20133" Ref="C42"  Part="1"
-F 0 "C42" H 9100 4550 50  0000 C CNN
+AR Path="/60B17C6E/60B20133" Ref="C36"  Part="1"
+F 0 "C36" H 9100 4550 50  0000 C CNN
 F 1 "0.1uF" H 9300 4700 50  0000 C CNN
 F 2 "Capacitor_SMD:C_0402_1005Metric" H 9150 4650 50  0001 C CNN
@@
 P 8550 4550
 AR Path="/60B2013A" Ref="#PWR?"  Part="1"
-AR Path="/60B17C6E/60B2013A" Ref="#PWR0158"  Part="1"
-F 0 "#PWR0158" H 8550 4400 50  0001 C CNN
+AR Path="/60B17C6E/60B2013A" Ref="#PWR067"  Part="1"
+F 0 "#PWR067" H 8550 4400 50  0001 C CNN
 F 1 "+3V3" H 8565 4723 50  0000 C CNN
 F 2 "" H 8550 4550 50  0001 C CNN
@@
 P 8550 4750
 AR Path="/60B20141" Ref="#PWR?"  Part="1"
-AR Path="/60B17C6E/60B20141" Ref="#PWR0159"  Part="1"
-F 0 "#PWR0159" H 8550 4500 50  0001 C CNN
+AR Path="/60B17C6E/60B20141" Ref="#PWR068"  Part="1"
+F 0 "#PWR068" H 8550 4500 50  0001 C CNN
 F 1 "GND" H 8650 4650 50  0000 C CNN
 F 2 "" H 8550 4750 50  0001 C CNN
@@
 P 7200 4200
 AR Path="/60B2014B" Ref="#PWR?"  Part="1"
-AR Path="/60B17C6E/60B2014B" Ref="#PWR0160"  Part="1"
-F 0 "#PWR0160" H 7200 3950 50  0001 C CNN
+AR Path="/60B17C6E/60B2014B" Ref="#PWR066"  Part="1"
+F 0 "#PWR066" H 7200 3950 50  0001 C CNN
 F 1 "GND" H 7300 4100 50  0000 C CNN
 F 2 "" H 7200 4200 50  0001 C CNN
@@
 P 7100 4100
 AR Path="/60B20154" Ref="R?"  Part="1"
-AR Path="/60B17C6E/60B20154" Ref="R34"  Part="1"
-F 0 "R34" V 7050 4200 50  0000 L CNN
+AR Path="/60B17C6E/60B20154" Ref="R18"  Part="1"
+F 0 "R18" V 7050 4200 50  0000 L CNN
 F 1 "75" V 7100 4050 50  0000 L CNN
 F 2 "Resistor_SMD:R_0402_1005Metric" H 7100 4100 50  0001 C CNN
@@
 P 8650 3000
 AR Path="/60B20160" Ref="#PWR?"  Part="1"
-AR Path="/60B17C6E/60B20160" Ref="#PWR0161"  Part="1"
-F 0 "#PWR0161" H 8650 2750 50  0001 C CNN
+AR Path="/60B17C6E/60B20160" Ref="#PWR063"  Part="1"
+F 0 "#PWR063" H 8650 2750 50  0001 C CNN
 F 1 "GND" H 8750 2900 50  0000 C CNN
 F 2 "" H 8650 3000 50  0001 C CNN
@@
 P 9000 2750
 AR Path="/60B20176" Ref="#PWR?"  Part="1"
-AR Path="/60B17C6E/60B20176" Ref="#PWR0162"  Part="1"
-F 0 "#PWR0162" H 9000 2600 50  0001 C CNN
+AR Path="/60B17C6E/60B20176" Ref="#PWR062"  Part="1"
+F 0 "#PWR062" H 9000 2600 50  0001 C CNN
 F 1 "+3V3" H 9015 2923 50  0000 C CNN
 F 2 "" H 9000 2750 50  0001 C CNN
@@
 P 6700 3150
 AR Path="/60B2017F" Ref="#PWR?"  Part="1"
-AR Path="/60B17C6E/60B2017F" Ref="#PWR0163"  Part="1"
-F 0 "#PWR0163" H 6700 3000 50  0001 C CNN
+AR Path="/60B17C6E/60B2017F" Ref="#PWR064"  Part="1"
+F 0 "#PWR064" H 6700 3000 50  0001 C CNN
 F 1 "+3V3" H 6715 3323 50  0000 C CNN
 F 2 "" H 6700 3150 50  0001 C CNN
@@
 P 8600 4150
 AR Path="/60B20185" Ref="#PWR?"  Part="1"
-AR Path="/60B17C6E/60B20185" Ref="#PWR0164"  Part="1"
-F 0 "#PWR0164" H 8600 3900 50  0001 C CNN
+AR Path="/60B17C6E/60B20185" Ref="#PWR065"  Part="1"
+F 0 "#PWR065" H 8600 3900 50  0001 C CNN
 F 1 "GND" H 8700 4050 50  0000 C CNN
 F 2 "" H 8600 4150 50  0001 C CNN
@@
 P 7900 3450
 AR Path="/60B20193" Ref="U?"  Part="1"
-AR Path="/60B17C6E/60B20193" Ref="U6"  Part="1"
-F 0 "U6" H 7900 4520 50  0000 C CNN
+AR Path="/60B17C6E/60B20193" Ref="U10"  Part="1"
+F 0 "U10" H 7900 4520 50  0000 C CNN
 F 1 "MAX7456EUI+" H 7900 4429 50  0000 C CNN
 F 2 "JPW_Footprints:MAX7456EUI&plus_T" H 7900 3450 50  0001 L BNN
@@
 P 8800 3450
 AR Path="/60B2019B" Ref="R?"  Part="1"
-AR Path="/60B17C6E/60B2019B" Ref="R30"  Part="1"
-F 0 "R30" V 8750 3550 50  0000 L CNN
+AR Path="/60B17C6E/60B2019B" Ref="R16"  Part="1"
+F 0 "R16" V 8750 3550 50  0000 L CNN
 F 1 "1k" V 8800 3400 50  0000 L CNN
 F 2 "Resistor_SMD:R_0402_1005Metric" H 8800 3450 50  0001 C CNN
@@
 P 8800 3250
 AR Path="/60B201A1" Ref="R?"  Part="1"
-AR Path="/60B17C6E/60B201A1" Ref="R29"  Part="1"
-F 0 "R29" V 8750 3350 50  0000 L CNN
+AR Path="/60B17C6E/60B201A1" Ref="R15"  Part="1"
+F 0 "R15" V 8750 3350 50  0000 L CNN
 F 1 "1k" V 8800 3200 50  0000 L CNN
 F 2 "Resistor_SMD:R_0402_1005Metric" H 8800 3250 50  0001 C CNN
@@
 P 8800 3150
 AR Path="/60B201A7" Ref="R?"  Part="1"
-AR Path="/60B17C6E/60B201A7" Ref="R25"  Part="1"
-F 0 "R25" V 8750 3250 50  0000 L CNN
+AR Path="/60B17C6E/60B201A7" Ref="R14"  Part="1"
+F 0 "R14" V 8750 3250 50  0000 L CNN
 F 1 "1k" V 8800 3100 50  0000 L CNN
 F 2 "Resistor_SMD:R_0402_1005Metric" H 8800 3150 50  0001 C CNN
@@
 P 9350 3750
 AR Path="/60B201AD" Ref="C?"  Part="1"
-AR Path="/60B17C6E/60B201AD" Ref="C38"  Part="1"
-F 0 "C38" V 9300 3650 50  0000 C CNN
+AR Path="/60B17C6E/60B201AD" Ref="C32"  Part="1"
+F 0 "C32" V 9300 3650 50  0000 C CNN
 F 1 "10uF" V 9400 3650 50  0000 C CNN
 F 2 "Capacitor_SMD:C_0402_1005Metric" H 9350 3750 50  0001 C CNN
@@
 P 9550 3650
 AR Path="/60B201B3" Ref="C?"  Part="1"
-AR Path="/60B17C6E/60B201B3" Ref="C37"  Part="1"
-F 0 "C37" V 9450 3700 50  0000 C CNN
+AR Path="/60B17C6E/60B201B3" Ref="C31"  Part="1"
+F 0 "C31" V 9450 3700 50  0000 C CNN
 F 1 "10uF" V 9500 3550 50  0000 C CNN
 F 2 "Capacitor_SMD:C_0402_1005Metric" H 9550 3650 50  0001 C CNN
@@
 P 9750 3650
 AR Path="/60B201BC" Ref="R?"  Part="1"
-AR Path="/60B17C6E/60B201BC" Ref="R33"  Part="1"
-F 0 "R33" V 9800 3700 50  0000 L CNN
+AR Path="/60B17C6E/60B201BC" Ref="R17"  Part="1"
+F 0 "R17" V 9800 3700 50  0000 L CNN
 F 1 "75" V 9750 3600 50  0000 L CNN
 F 2 "Resistor_SMD:R_0402_1005Metric" H 9750 3650 50  0001 C CNN
@@
 P 7100 3900
 AR Path="/60B201C2" Ref="C?"  Part="1"
-AR Path="/60B17C6E/60B201C2" Ref="C39"  Part="1"
-F 0 "C39" V 7150 3800 50  0000 C CNN
+AR Path="/60B17C6E/60B201C2" Ref="C33"  Part="1"
+F 0 "C33" V 7150 3800 50  0000 C CNN
 F 1 "0.1uF" V 7150 4050 50  0000 C CNN
 F 2 "Capacitor_SMD:C_0402_1005Metric" H 7100 3900 50  0001 C CNN
@@
 Text Notes 5000 1800 0    591  ~ 118
 OSD
+Text Label 8600 3150 1    50   ~ 0
+HSYNC
+Text Label 8700 3250 1    50   ~ 0
+LSYNC
+Text Label 8600 3450 0    50   ~ 0
+LOS
+Text Label 8600 3650 0    50   ~ 0
+VOUT
+Text Label 7200 3750 2    50   ~ 0
+VIN
 $EndSCHEMATC

Commit message: Changes made
Parts:
- renumbered C31 to C29, C32 to C30, C33 to C31, C34 to C32, C35 to C33, C36 to C34, C37 to C35, C38 to C36, U10 to U9
Changed lines of the file:
@@
 P 7200 4850
 AR Path="/60B200F8" Ref="C?"  Part="1"
-AR Path="/60B17C6E/60B200F8" Ref="C37"  Part="1"
-F 0 "C37" H 7350 4800 50  0000 R CNN
+AR Path="/60B17C6E/60B200F8" Ref="C35"  Part="1"
+F 0 "C35" H 7350 4800 50  0000 R CNN
 F 1 "10pF" H 7500 4900 50  0000 R CNN
 F 2 "Capacitor_SMD:C_0402_1005Metric" H 7200 4850 50  0001 C CNN
@@
 P 7600 4850
 AR Path="/60B20102" Ref="C?"  Part="1"
-AR Path="/60B17C6E/60B20102" Ref="C38"  Part="1"
-F 0 "C38" H 7550 4800 50  0000 R CNN
+AR Path="/60B17C6E/60B20102" Ref="C36"  Part="1"
+F 0 "C36" H 7550 4800 50  0000 R CNN
 F 1 "10pF" H 7500 4900 50  0000 R CNN
 F 2 "Capacitor_SMD:C_0402_1005Metric" H 7600 4850 50  0001 C CNN
@@
 P 7350 4950
 AR Path="/60B2010C" Ref="#PWR?"  Part="1"
-AR Path="/60B17C6E/60B2010C" Ref="#PWR069"  Part="1"
-F 0 "#PWR069" H 7350 4700 50  0001 C CNN
+AR Path="/60B17C6E/60B2010C" Ref="#PWR063"  Part="1"
+F 0 "#PWR063" H 7350 4700 50  0001 C CNN
 F 1 "GND" H 7355 4777 50  0000 C CNN
 F 2 "" H 7350 4950 50  0001 C CNN
@@
 P 8550 4650
 AR Path="/60B20121" Ref="C?"  Part="1"
-AR Path="/60B17C6E/60B20121" Ref="C34"  Part="1"
-F 0 "C34" H 8400 4550 50  0000 C CNN
+AR Path="/60B17C6E/60B20121" Ref="C32"  Part="1"
+F 0 "C32" H 8400 4550 50  0000 C CNN
 F 1 "0.1uF" H 8650 4700 50  0000 C CNN
 F 2 "Capacitor_SMD:C_0402_1005Metric" H 8550 4650 50  0001 C CNN
@@
 P 8850 4650
 AR Path="/60B20127" Ref="C?"  Part="1"
-AR Path="/60B17C6E/60B20127" Ref="C35"  Part="1"
-F 0 "C35" H 8750 4550 50  0000 C CNN
+AR Path="/60B17C6E/60B20127" Ref="C33"  Part="1"
+F 0 "C33" H 8750 4550 50  0000 C CNN
 F 1 "0.1uF" H 9000 4700 50  0000 C CNN
 F 2 "Capacitor_SMD:C_0402_1005Metric" H 8850 4650 50  0001 C CNN
@@
 P 9150 4650
 AR Path="/60B20133" Ref="C?"  Part="1"
-AR Path="/60B17C6E/60B20133" Ref="C36"  Part="1"
-F 0 "C36" H 9100 4550 50  0000 C CNN
+AR Path="/60B17C6E/60B20133" Ref="C34"  Part="1"
+F 0 "C34" H 9100 4550 50  0000 C CNN
 F 1 "0.1uF" H 9300 4700 50  0000 C CNN
 F 2 "Capacitor_SMD:C_0402_1005Metric" H 9150 4650 50  0001 C CNN
@@
 P 8550 4550
 AR Path="/60B2013A" Ref="#PWR?"  Part="1"
-AR Path="/60B17C6E/60B2013A" Ref="#PWR067"  Part="1"
-F 0 "#PWR067" H 8550 4400 50  0001 C CNN
+AR Path="/60B17C6E/60B2013A" Ref="#PWR061"  Part="1"
+F 0 "#PWR061" H 8550 4400 50  0001 C CNN
 F 1 "+3V3" H 8565 4723 50  0000 C CNN
 F 2 "" H 8550 4550 50  0001 C CNN
@@
 P 8550 4750
 AR Path="/60B20141" Ref="#PWR?"  Part="1"
-AR Path="/60B17C6E/60B20141" Ref="#PWR068"  Part="1"
-F 0 "#PWR068" H 8550 4500 50  0001 C CNN
+AR Path="/60B17C6E/60B20141" Ref="#PWR062"  Part="1"
+F 0 "#PWR062" H 8550 4500 50  0001 C CNN
 F 1 "GND" H 8650 4650 50  0000 C CNN
 F 2 "" H 8550 4750 50  0001 C CNN
@@
 P 7200 4200
 AR Path="/60B2014B" Ref="#PWR?"  Part="1"
-AR Path="/60B17C6E/60B2014B" Ref="#PWR066"  Part="1"
-F 0 "#PWR066" H 7200 3950 50  0001 C CNN
+AR Path="/60B17C6E/60B2014B" Ref="#PWR060"  Part="1"
+F 0 "#PWR060" H 7200 3950 50  0001 C CNN
 F 1 "GND" H 7300 4100 50  0000 C CNN
 F 2 "" H 7200 4200 50  0001 C CNN
@@
 P 8650 3000
 AR Path="/60B20160" Ref="#PWR?"  Part="1"
-AR Path="/60B17C6E/60B20160" Ref="#PWR063"  Part="1"
-F 0 "#PWR063" H 8650 2750 50  0001 C CNN
+AR Path="/60B17C6E/60B20160" Ref="#PWR057"  Part="1"
+F 0 "#PWR057" H 8650 2750 50  0001 C CNN
 F 1 "GND" H 8750 2900 50  0000 C CNN
 F 2 "" H 8650 3000 50  0001 C CNN
@@
 P 9000 2750
 AR Path="/60B20176" Ref="#PWR?"  Part="1"
-AR Path="/60B17C6E/60B20176" Ref="#PWR062"  Part="1"
-F 0 "#PWR062" H 9000 2600 50  0001 C CNN
+AR Path="/60B17C6E/60B20176" Ref="#PWR056"  Part="1"
+F 0 "#PWR056" H 9000 2600 50  0001 C CNN
 F 1 "+3V3" H 9015 2923 50  0000 C CNN
 F 2 "" H 9000 2750 50  0001 C CNN
@@
 P 6700 3150
 AR Path="/60B2017F" Ref="#PWR?"  Part="1"
-AR Path="/60B17C6E/60B2017F" Ref="#PWR064"  Part="1"
-F 0 "#PWR064" H 6700 3000 50  0001 C CNN
+AR Path="/60B17C6E/60B2017F" Ref="#PWR058"  Part="1"
+F 0 "#PWR058" H 6700 3000 50  0001 C CNN
 F 1 "+3V3" H 6715 3323 50  0000 C CNN
 F 2 "" H 6700 3150 50  0001 C CNN
@@
 P 8600 4150
 AR Path="/60B20185" Ref="#PWR?"  Part="1"
-AR Path="/60B17C6E/60B20185" Ref="#PWR065"  Part="1"
-F 0 "#PWR065" H 8600 3900 50  0001 C CNN
+AR Path="/60B17C6E/60B20185" Ref="#PWR059"  Part="1"
+F 0 "#PWR059" H 8600 3900 50  0001 C CNN
 F 1 "GND" H 8700 4050 50  0000 C CNN
 F 2 "" H 8600 4150 50  0001 C CNN
@@
 P 7900 3450
 AR Path="/60B20193" Ref="U?"  Part="1"
-AR Path="/60B17C6E/60B20193" Ref="U10"  Part="1"
-F 0 "U10" H 7900 4520 50  0000 C CNN
+AR Path="/60B17C6E/60B20193" Ref="U9"  Part="1"
+F 0 "U9" H 7900 4520 50  0000 C CNN
 F 1 "MAX7456EUI+" H 7900 4429 50  0000 C CNN
 F 2 "JPW_Footprints:MAX7456EUI&plus_T" H 7900 3450 50  0001 L BNN
@@
 P 9350 3750
 AR Path="/60B201AD" Ref="C?"  Part="1"
-AR Path="/60B17C6E/60B201AD" Ref="C32"  Part="1"
-F 0 "C32" V 9300 3650 50  0000 C CNN
+AR Path="/60B17C6E/60B201AD" Ref="C30"  Part="1"
+F 0 "C30" V 9300 3650 50  0000 C CNN
 F 1 "10uF" V 9400 3650 50  0000 C CNN
 F 2 "Capacitor_SMD:C_0402_1005Metric" H 9350 3750 50  0001 C CNN
@@
 P 9550 3650
 AR Path="/60B201B3" Ref="C?"  Part="1"
-AR Path="/60B17C6E/60B201B3" Ref="C31"  Part="1"
-F 0 "C31" V 9450 3700 50  0000 C CNN
+AR Path="/60B17C6E/60B201B3" Ref="C29"  Part="1"
+F 0 "C29" V 9450 3700 50  0000 C CNN
 F 1 "10uF" V 9500 3550 50  0000 C CNN
 F 2 "Capacitor_SMD:C_0402_1005Metric" H 9550 3650 50  0001 C CNN
@@
 P 7100 3900
 AR Path="/60B201C2" Ref="C?"  Part="1"
-AR Path="/60B17C6E/60B201C2" Ref="C33"  Part="1"
-F 0 "C33" V 7150 3800 50  0000 C CNN
+AR Path="/60B17C6E/60B201C2" Ref="C31"  Part="1"
+F 0 "C31" V 7150 3800 50  0000 C CNN
 F 1 "0.1uF" V 7150 4050 50  0000 C CNN
 F 2 "Capacitor_SMD:C_0402_1005Metric" H 7100 3900 50  0001 C CNN
