File: Power.sch (KiCad schematic (older format))
At the start: 38 parts, among them U1 LP2985-3.3, U3 LP2985-3.3, U4 MP4560_QFN10, U5 MP4560_QFN10

Commit message: Lots of changes made
Parts:
- removed C1: 1uF, Capacitor_SMD:C_0402_1005Metric, symbol Device:C_Small
- removed C16: 2.2uF, Capacitor_SMD:C_0402_1005Metric, symbol Device:C_Small
- removed C2: 10nF, Capacitor_SMD:C_0402_1005Metric, symbol Device:C_Small
- removed U1, U3: LP2985-3.3, Package_TO_SOT_SMD:SOT-23-5, symbol Regulator_Linear:LP2985-3.3
- removed U4, U5: MP4560_QFN10, Package_DFN_QFN:DFN-10-1EP_3x3mm_P0.5mm_EP1.7x2.5mm, symbol Regulator_Switching:MP4560_QFN10
- added C13, C14: 10uF, Capacitor_SMD:C_0402_1005Metric, symbol Device:C_Small
- added U1, U2: MP4462, Package_DFN_QFN:DFN-10-1EP_3x3mm_P0.5mm_EP1.7x2.5mm, symbol Regulator_Switching:MP4462
- added U3: LD1086DT33TR, Package_TO_SOT_SMD:TO-252-2, symbol Regulator_Linear:LD1086DT33TR
- added U4: LP2985-1.8, Package_TO_SOT_SMD:SOT-23-5, symbol Regulator_Linear:LP2985-1.8
- C10: renamed from C34; value 390pF -> 330pF
- C3: renamed from C23; value 22uF -> 33uF; footprint Capacitor_SMD:C_0603_1608Metric -> Capacitor_SMD:C_0402_1005Metric
- C4: renamed from C22; footprint Capacitor_SMD:C_0603_1608Metric -> Capacitor_SMD:C_0402_1005Metric
- C5: renamed from C29; footprint Capacitor_SMD:C_0603_1608Metric -> Capacitor_SMD:C_0402_1005Metric
- C7: renamed from C24; footprint Capacitor_SMD:C_0603_1608Metric -> Capacitor_SMD:C_0402_1005Metric
- C9: renamed from C33; value 390pF -> 330pF
- L4: renamed from L2; value 12uH -> 6.8uH
- L5: renamed from L1; value 15uH -> 8.2uH
- R7: renamed from R24; value 93.1k -> 127k
- R8: renamed from R22; value 165k -> 147k
- renumbered C21 to C1, C35 to C11, C36 to C12, C17 to C15, C18 to C16, C19 to C17, C20 to C2, C31 to C6, C28 to C8, D6 to D1, D4 to D2, D1 to D3, D2 to D4, FB3 to FB2, R11 to R1, R10 to R2, R13 to R3, R12 to R4, R19 to R5, R17 to R6
Connections:
- net labels added: +1V8, +4V5, BP_1V8, BS_5, BS_9, COMP_5, COMP_9, FB_5, FB_9, FREQ_5, FREQ_9, SW_5, SW_9, VIN_1V8, VIN_3V3
- net labels removed: +3V3_GYRO, 4V5
- wire segments 101 -> 93

Commit message: Increased board size and added silkscreen text
Parts:
- D3, D4: footprint Footprints:SBR3U30P1-7 -> Diode_SMD:D_SOD-123F
Changed lines of the file:
@@
 F 1 "90V, 2A" V 3400 1100 50  0000 L CNN
 F 2 "Diode_SMD:D_SOD-123F" V 3300 1300 50  0001 C CNN
-F 3 "~" V 3300 1300 50  0001 C CNN
+F 3 "MBR230S1F-7" V 3300 1300 50  0001 C CNN
 	1    3300 1300
 	0    1    1    0
@@
 F 1 "90V, 2A" V 9350 1050 50  0000 L CNN
 F 2 "Diode_SMD:D_SOD-123F" V 9250 1250 50  0001 C CNN
-F 3 "~" V 9250 1250 50  0001 C CNN
+F 3 "MBR230S1F-7" V 9250 1250 50  0001 C CNN
 	1    9250 1250
 	0    1    1    0
@@
 F 0 "D3" H 7650 5183 50  0000 C CNN
 F 1 "D_Schottky" H 7650 5274 50  0000 C CNN
-F 2 "Footprints:SBR3U30P1-7" H 7650 5400 50  0001 C CNN
-F 3 "~" H 7650 5400 50  0001 C CNN
+F 2 "Diode_SMD:D_SOD-123F" H 7650 5400 50  0001 C CNN
+F 3 "MBR230S1F-7" H 7650 5400 50  0001 C CNN
 	1    7650 5400
 	-1   0    0    1
@@
 F 0 "D4" H 7650 5483 50  0000 C CNN
 F 1 "D_Schottky" H 7650 5574 50  0000 C CNN
-F 2 "Footprints:SBR3U30P1-7" H 7650 5700 50  0001 C CNN
-F 3 "~" H 7650 5700 50  0001 C CNN
+F 2 "Diode_SMD:D_SOD-123F" H 7650 5700 50  0001 C CNN
+F 3 "MBR230S1F-7" H 7650 5700 50  0001 C CNN
 	1    7650 5700
 	-1   0    0    1

Commit message: Changes made
Parts:
- removed U4: LP2985-1.8, Package_TO_SOT_SMD:SOT-23-5, symbol Regulator_Linear:LP2985-1.8
- added U4: LP2985-3.3, Package_TO_SOT_SMD:SOT-23-5, symbol Regulator_Linear:LP2985-3.3
- renumbered L4 to L3, L5 to L4
Connections:
- net BP_1V8: now also U4.4 (BP)
- net GND: now also U4.2 (GND)
- net VIN_1V8: now also U4.1 (VIN), U4.3 (ON/~OFF~)
- net +1V8 renamed +3V3_GYRO
- net +3V3_GYRO: now also U4.5 (VOUT)
Changed lines of the file:
@@
 P 3450 1200
 AR Path="/609679E1" Ref="L?"  Part="1"
-AR Path="/6094AC2B/609679E1" Ref="L5"  Part="1"
-F 0 "L5" V 3635 1200 50  0000 C CNN
+AR Path="/6094AC2B/609679E1" Ref="L4"  Part="1"
+F 0 "L4" V 3635 1200 50  0000 C CNN
 F 1 "8.2uH" V 3544 1200 50  0000 C CNN
 F 2 "Inductor_SMD:L_Bourns-SRN3015" H 3450 1200 50  0001 C CNN
@@
 P 9400 1150
 AR Path="/60967B08" Ref="L?"  Part="1"
-AR Path="/6094AC2B/60967B08" Ref="L4"  Part="1"
-F 0 "L4" V 9585 1150 50  0000 C CNN
+AR Path="/6094AC2B/60967B08" Ref="L3"  Part="1"
+F 0 "L3" V 9585 1150 50  0000 C CNN
 F 1 "6.8uH" V 9494 1150 50  0000 C CNN
 F 2 "Inductor_SMD:L_Bourns-SRN3015" H 9400 1150 50  0001 C CNN
@@
 	1    0    0    -1
 $EndComp
-$Comp
-L Regulator_Linear:LP2985-1.8 U4
-U 1 1 61821DAA
-P 5250 5500
-F 0 "U4" H 5250 5842 50  0000 C CNN
-F 1 "LP2985-1.8" H 5250 5751 50  0000 C CNN
-F 2 "Package_TO_SOT_SMD:SOT-23-5" H 5250 5825 50  0001 C CNN
-F 3 "http://www.ti.com/lit/ds/symlink/lp2985.pdf" H 5250 5500 50  0001 C CNN
-	1    5250 5500
-	1    0    0    -1
-$EndComp
 Wire Wire Line
 	5650 5400 6000 5400
-$Comp
-L power:+1V8 #PWR024
-U 1 1 61826B78
-P 6000 5400
-F 0 "#PWR024" H 6000 5250 50  0001 C CNN
-F 1 "+1V8" H 6015 5573 50  0000 C CNN
-F 2 "" H 6000 5400 50  0001 C CNN
-F 3 "" H 6000 5400 50  0001 C CNN
-	1    6000 5400
-	1    0    0    -1
-$EndComp
-Connection ~ 6000 5400
 Text Label 2150 1800 2    50   ~ 0
 FREQ_9
@@
 Text Label 2700 5400 1    50   ~ 0
 VIN_3V3
+$Comp
+L Regulator_Linear:LP2985-3.3 U4
+U 1 1 6191D328
+P 5250 5500
+F 0 "U4" H 5250 5842 50  0000 C CNN
+F 1 "LP2985-3.3" H 5250 5751 50  0000 C CNN
+F 2 "Package_TO_SOT_SMD:SOT-23-5" H 5250 5825 50  0001 C CNN
+F 3 "http://www.ti.com/lit/ds/symlink/lp2985.pdf" H 5250 5500 50  0001 C CNN
+	1    5250 5500
+	1    0    0    -1
+$EndComp
+$Comp
+L power:+3V3_GYRO #PWR0125
+U 1 1 6191FD25
+P 6000 5400
+F 0 "#PWR0125" H 6000 5250 50  0001 C CNN
+F 1 "+3V3_GYRO" H 6015 5573 50  0000 C CNN
+F 2 "" H 6000 5400 50  0001 C CNN
+F 3 "" H 6000 5400 50  0001 C CNN
+	1    6000 5400
+	1    0    0    -1
+$EndComp
+Connection ~ 6000 5400
 $EndSCHEMATC
