File: Autodrone.kicad_pcb (KiCad board)
At the start: 6 copper layers, 54.8 x 39.2 mm, 143 parts, among them J1 Conn_01x03, J10 Conn_01x03, J11 Conn_01x02, J12 Conn_01x03, J13 Conn_01x02, J14 Conn_01x04, J15 Conn_01x04, J16 Conn_01x03, J17 Conn_01x03, J2 USB_B_Micro, J3 Conn_01x08, J4 Conn_01x08, J5 Conn_01x04, J6 Conn_01x02, J7 Conn_01x02, J8 Conn_01x04, J9 Conn_01x04, Q1 BSS138, SW1 SW_Push, U1 MP4462, U10 MAX7456EUI+, U11 STM32F722RETx, U2 MP4462, U3 LD1086DT33TR, U4 LP2985-1.8, U5 SN74AXC4T774BQBR, U6 ICM-20948, U7 BMP280, U8 DRV8424E, U9 STLINK-V3MODS, Y1 27MHz, Y2 CSTNE8M00G55Z000R0

Commit message: Changes made
Parts:
- removed the C21 at (97.5, 90.7)
- removed the C22 at (99.4, 88.8)
- removed the U6 at (100.3, 91.6)
- added L5: LED, Footprints:LED, F.Cu at (78.0, 101.2)
- added L6: LED, Footprints:LED, F.Cu at (76.7, 79.0)
- C19: value 0.1uF -> 2.2nF
- L1: renamed from L2; moved to F.Cu
- U4: value LP2985-1.8 -> LP2985-3.3
- U5: value SN74AXC4T774BQBR -> MPU-6000; footprint Footprints:SN74AXC4T774BQBR -> Sensor_Motion:InvenSense_QFN-24_4x4mm_P0.5mm
- moved L1 23.4 mm to (111.3, 99.0), turned to 90 degrees
- moved C19 7.81 mm to (98.5, 96.0), turned to 180 degrees
- moved C20 5.17 mm to (99.5, 89.2)
- moved C18 5.16 mm to (97.1, 90.0), turned to 90 degrees
- moved U5 3.03 mm to (100.2, 92.6), turned to 180 degrees
- moved C32 1.24 mm to (104.1, 90.4), turned to 90 degrees
- moved L2 0.44 mm to (104.7, 95.5)
- moved U4 0.14 mm to (100.0, 86.3)
- renumbered C23 to C21, C24 to C22, C25 to C23, C26 to C24, C27 to C25, C28 to C26, C29 to C27, C30 to C28, C31 to C29, C32 to C30, C33 to C31, C34 to C32, C35 to C33, C36 to C34, C37 to C35, C38 to C36, C39 to C37, C40 to C38, C41 to C39, C42 to C40, C43 to C41, C44 to C42, C45 to C43, C46 to C44, C47 to C45, C48 to C46, J8 to J1, J6 to J10, J7 to J11, J10 to J12, J16 to J13, J11 to J14, J12 to J15, J13 to J16, J9 to J2, J1 to J3, J2 to J4, J3 to J5, J4 to J6, J14 to J7, J15 to J8, J5 to J9, L3 to L2, L4 to L3, L5 to L4, U11 to U10, U7 to U6, U8 to U7, U9 to U8, U10 to U9
Connections:
- net /MCU/1V8 renamed /MCU/3V3_GYRO
- C17 pad 1: +1V8 -> +3V3_GYRO
- C18 pad 1: +3V3 -> +3V3_GYRO
- C19 pad 1: +1V8 -> /Gyro/CPOUT
- C20 pad 1: +1V8 -> /Gyro/REGOUT
- D6 pad 2: +1V8 -> +3V3_GYRO
- U10 pad 20: /MCU/SPI1_CS -> /Gyro/SPI1_CS
- U10 pad 21: /Gyro/SPI1_MISO -> /Gyro/SPI1_SCK
- U10 pad 22: /MCU/SPI1_MISO -> /Gyro/SPI1_MISO
- U10 pad 23: /Gyro/SPI1_CS -> /Gyro/SPI1_MOSI
- U4 pad 5: +1V8 -> +3V3_GYRO
- U5 pad 1: /Gyro/SPI1_CS -> GND
- U5 pad 10: /Gyro/ICM_MOSI -> /Gyro/REGOUT
- U5 pad 11: /Gyro/ICM_SCK -> GND
- U5 pad 12: /Gyro/ICM_CS -> (no net)
- U5 pad 13: +1V8 -> +3V3_GYRO
- U5 pad 14: +3V3 -> (no net)
- U5 pad 15: +3V3 -> (no net)
- U5 pad 16: +3V3 -> (no net)
- U5 pad 2: /MCU/SPI1_MISO -> (no net)
- U5 pad 3: /MCU/SPI1_CS -> (no net)
- U5 pad 4: /Gyro/SPI1_MISO -> (no net)
- U5 pad 5: +3V3 -> (no net)
- U5 pad 6: GND -> (no net)
- U5 pad 7: GND -> (no net)
- U5 pad 8: GND -> /Gyro/SPI1_CS
- U5 pad 9: /Gyro/ICM_MISO -> /Gyro/SPI1_MISO
Routing:
- net +1V8: track 52.9 -> 0.00 mm, vias 2 -> 0
- net +3V3_GYRO: track 0.00 -> 39.7 mm
- net /MCU/SPI1_CS: track 17.0 -> 0.00 mm, vias 2 -> 0
- net /MCU/SPI1_MISO: track 16.7 -> 0.00 mm, vias 2 -> 0
- net /Gyro/SPI1_CS: track 18.2 -> 6.43 mm, vias 2 -> 1
- net /Gyro/SPI1_SCK: track 0.00 -> 11.3 mm, vias 0 -> 1
- net /Gyro/ICM_MISO: track 11.0 -> 0.00 mm
- net /Gyro/SPI1_MOSI: track 0.00 -> 8.31 mm, vias 0 -> 1
- net /Gyro/SPI1_MISO: track 14.5 -> 7.14 mm, vias 2 -> 1
- net +3V3: track 67.2 -> 60.7 mm
- net /Gyro/CPOUT: track 0.00 -> 1.62 mm
- net /Gyro/ICM_MOSI: track 1.54 -> 0.00 mm
- net /Gyro/ICM_SCK: track 1.50 -> 0.00 mm
- net /Gyro/ICM_CS: track 1.46 -> 0.00 mm
- net /Connectors/I2C2_SDA: track 36.8 -> 38.2 mm
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Other:
- board text added: "VCC +9V +5V 3V3 GYRO"
- board text removed: "VCC +9V +5V 3V3 1V8"
